File: BreakoutBoards/IMUBreakout/IMUBreakout.kicad_pcb (KiCad board)
At the start: 2 copper layers, 23.3 x 18.9 mm, 18 parts, among them J10 IMU Connection, J5 Qwicc, U1 ICM-20948, U2 MIC5504-1.8YM5

Commit message: update pcb
Parts:
- removed the ? at (153.6, 77.4)
- removed the ? at (153.6, 63.9)
- removed the ? at (172.2, 63.9)
- removed the ? at (172.2, 77.4)
- added ?: , , F.Cu at (153.6, 77.4)
- added ?: , , F.Cu at (153.6, 64.0)
- added ?: , , F.Cu at (172.2, 77.4)
- added ?: , , F.Cu at (172.2, 64.0)
- added G***: LOGO, LOGO, B.Cu at (163.0, 70.6)
- added G***: LOGO, SparkFun-Qwiic:qwiic_4mm, B.Cu at (154.2, 70.7)
- moved C5 2.08 mm to (163.2, 74.3), turned to 0 degrees
- moved C6 0.50 mm to (160.4, 68.5)
- moved C7 0.48 mm to (160.4, 72.6)
Connections:
- U1 pad 22: unconnected-(U1-~{CS}-Pad22) -> +1V8
Routing:
- net +3V3: track 0.00 -> 40.3 mm
- net +1V8: track 0.00 -> 33.2 mm, vias 0 -> 3
- net /SCL: track 0.00 -> 18.3 mm, vias 0 -> 2
- net /SDA: track 0.00 -> 17.3 mm, vias 0 -> 3
- net /INT1: track 0.00 -> 12.6 mm, vias 0 -> 2
- net /AD0: track 0.00 -> 10.2 mm
- net Earth: track 0.00 -> 7.85 mm, vias 0 -> 50
- net Net-(U1-REGOUT): track 0.00 -> 1.61 mm
- added copper zone on B.Cu, net Earth
- added copper zone on F.Cu, net Earth
Other:
- board text added: "ICM 20948"
- board text added: "ICM-20948 Breakout"
- board text added: "Max Kendall W0MXX"

Commit message: updated IMU board and production files
Parts:
- removed ? (x4): , 
- removed C3, C4: 1uF, Capacitor_SMD:C_0603_1608Metric
- removed C7: 100nF, Capacitor_SMD:C_0603_1608Metric
- removed U2: MIC5504-1.8YM5, Package_TO_SOT_SMD:SOT-23-5
- added G***: LOGO, LOGO, F.Cu at (150.6, 89.3)
- added H1: MountingHole, MountingHole:MountingHole_2.2mm_M2_Pad_Via, F.Cu at (158.4, 90.8)
- added H2: MountingHole, MountingHole:MountingHole_2.2mm_M2_Pad_Via, F.Cu at (141.8, 90.8)
- added J11: Dev Headers, Connector_PinSocket_2.54mm:PinSocket_1x06_P2.54mm_Vertical, F.Cu at (143.8, 105.0)
- C1, C2, C5, C6: footprint Capacitor_SMD:C_0603_1608Metric -> Capacitor_SMD:C_0402_1005Metric
- G***: moved to F.Cu
- R1, R2: footprint Resistor_SMD:R_0603_1608Metric -> Resistor_SMD:R_0402_1005Metric
- U1: value ICM-20948 -> ICM-42607-P; footprint Sensor_Motion:InvenSense_QFN-24_3x3mm_P0.4mm -> Package_LGA:Bosch_LGA-14_3x2.5mm_P0.5mm
- moved G*** 33.9 mm to (142.7, 102.5), turned to 0 degrees
- moved R2 32.7 mm to (154.7, 99.2), turned to 90 degrees
- moved C1 31.3 mm to (145.1, 97.4)
- moved J10 30.5 mm to (158.7, 98.3)
- moved J5 30.5 mm to (141.4, 98.3)
- moved C6 29.2 mm to (147.9, 94.8)
- moved C2 29.0 mm to (154.7, 101.2)
- moved R1 28.2 mm to (154.7, 97.3), turned to -90 degrees
- moved U1 28.1 mm to (150.0, 96.1)
- moved G*** 27.7 mm to (149.9, 95.0)
- moved C5 27.5 mm to (147.9, 97.2), turned to 90 degrees
- moved JP1 27.1 mm to (150.1, 100.6)
Connections:
- C6 pad 1: +1V8 -> +3V3
- J10 pad 5: /INT1 -> /INT2
- J10 pad 6: /INT2 -> /INT1
- JP1 pad 3: +1V8 -> +3V3
- R1 pad 2: /SDA -> /SCL
- R2 pad 2: /SCL -> /SDA
- U1 pad 1: unconnected-(U1-NC-Pad1) -> /AD0
- U1 pad 10: Net-(U1-REGOUT) -> unconnected-(U1-RESV-Pad10)
- U1 pad 11: Earth -> unconnected-(U1-RESV-Pad11)
- U1 pad 12: /INT1 -> +3V3
- U1 pad 13: +3V3 -> /SCL
- U1 pad 14: unconnected-(U1-NC-Pad14) -> /SDA
- U1 pad 4: unconnected-(U1-NC-Pad4) -> /INT1
- U1 pad 5: unconnected-(U1-NC-Pad5) -> +3V3
- U1 pad 6: unconnected-(U1-NC-Pad6) -> Earth
- U1 pad 7: unconnected-(U1-AUX_CL-Pad7) -> Earth
- U1 pad 8: +1V8 -> +3V3
- U1 pad 9: /AD0 -> /INT2
Routing:
- net +1V8: track 33.2 -> 0.00 mm, vias 3 -> 0
- net /INT2: track 0.00 -> 21.1 mm, vias 0 -> 1
- net /SCL: track 18.3 -> 30.9 mm, vias 2 -> 0
- net /INT1: track 12.6 -> 20.6 mm, vias 2 -> 0
- net /AD0: track 10.2 -> 17.8 mm, vias 0 -> 2
- net /SDA: track 17.3 -> 24.9 mm, vias 3 -> 2
- net Net-(U1-REGOUT): track 1.61 -> 0.00 mm
- net +3V3: track 40.3 -> 38.7 mm, vias 0 -> 7
- net Earth: track 7.85 -> 7.40 mm, vias 50 -> 41
Other:
- board size 23.3 x 18.9 mm -> 23.3 x 20.9 mm
- board text added: "0x68"
- board text added: "0x69"
- board text added: "ICM-42607-P Module"
- board text added: "IMU Module"
- board text removed: "0x68 0x69"
- board text removed: "ICM 20948"
- board text removed: "ICM-20948 Breakout"
